File: pcbs/InternalPCBV2/Display-RTC.kicad_sch (KiCad schematic)
At the start: 0 parts

Commit message: Neue Datei für Display & RTC Chip(s)
Parts:
- added BT1: Battery, symbol Device:Battery
- added C8: 0.1u, Capacitor_SMD:C_0402_1005Metric, symbol Device:C
- added R10, R11, R9: 10k, Capacitor_SMD:C_0402_1005Metric, symbol Device:R
- added U4: DS3231M, Package_SO:SOIC-16W_7.5x10.3mm_P1.27mm, symbol Timer_RTC:DS3231M
Connections:
- new net: BT1.1 (+), U4.14 (VBAT)
- new net +3.3V: C8.1, R10.1, R11.1, R9.1, U4.2 (VCC)
- new net GND: BT1.2 (-), C8.2, U4.10 (GND), U4.11 (GND), U4.12 (GND), U4.13 (GND), U4.5 (GND), U4.6 (GND), U4.7 (GND), U4.8 (GND), U4.9 (GND)
- new net I2C0_SCL: R9.2, U4.16 (SCL)
- new net I2C0_SDA: R10.2, U4.15 (SDA)
- new net RTC_IRQ: R11.2, U4.3 (~{INT}/SQW)
- no-connect marks 0 -> 2

Commit message: Neuer Footprint für MH-Z19B/C CO2 Sensor
Parts:
- added U5: ~, Display:Pico-ResTouch-LCD-2.8, symbol Display_Graphic:Pico-ResTouch-LCD-2.8
- BT1: footprint (none) -> Battery:BatteryHolder_Keystone_103_1x20mm
- R10, R11, R9: footprint Capacitor_SMD:C_0402_1005Metric -> Resistor_SMD:R_0402_1005Metric
Connections:
- net GND: now also U5.3 (GND)
- new net +5V: U5.39 (VCC)
- new net DISPLAY_BL: U5.17 (LCD_BL)
- new net DISPLAY_CS: U5.12 (LCD_CS)
- new net DISPLAY_DC: U5.11 (LCD_DC)
- new net DISPLAY_RST: U5.20 (LCD_RST)
- new net SDIO_CLK: U5.7 (SDIO_CLK)
- new net SDIO_CMD: U5.24 (SDIO_CMD)
- new net SDIO_D0: U5.25 (SDIO_D0)
- new net SDIO_D1: U5.26 (SDIO_D1)
- new net SDIO_D2: U5.27 (SDIO_D2)
- new net SDIO_D3CS: U5.29 (SDIO_CSD3)
- new net SPI1_RX: U5.16 (MISO)
- new net SPI1_SCK: U5.14 (LCD_CLK)
- new net SPI1_TX: U5.15 (MOSI)
- new net TP_CS: U5.21 (TP_CS)
- new net TP_IRQ: U5.22 (TP_IRQ)
Other:
- note added: "Sind TX und RX richtig herum?"
Changed lines of the file:
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@@
   (title_block
     (title "Innenmodul V2")
-    (date "2024-01-28")
+    (date "2024-01-31")
     (rev "A")
     (company "HAW Hamburg")
-    (comment 1 "Lasse Kelling")
+    (comment 1 "Lasse Kelling, Fabian Schmalenbach")
     (comment 2 "Display und RTC")
   )
@@
     (stroke (width 0) (type default))
   )
+  (text "Sind TX und RX richtig herum?" (at 151.13 106.68 0)
+    (effects (font (size 1.27 1.27)) (justify left bottom))
+  )
+  (label "SPI1_RX" (at 180.34 100.33 180) (fields_autoplaced)
+    (effects (font (size 1.27 1.27)) (justify right bottom))
+  )
+  (label "SDIO_D2" (at 215.9 90.17 0) (fields_autoplaced)
+    (effects (font (size 1.27 1.27)) (justify left bottom))
+  )
+  (label "SDIO_D1" (at 215.9 87.63 0) (fields_autoplaced)
+    (effects (font (size 1.27 1.27)) (justify left bottom))
+  )
+  (label "SPI1_TX" (at 180.34 97.79 180) (fields_autoplaced)
+    (effects (font (size 1.27 1.27)) (justify right bottom))
+  )
   (label "RTC_IRQ" (at 69.85 48.26 0) (fields_autoplaced)
     (effects (font (size 1.27 1.27)) (justify left bottom))
   )
+  (label "SDIO_CLK" (at 215.9 80.01 0) (fields_autoplaced)
+    (effects (font (size 1.27 1.27)) (justify left bottom))
+  )
+  (label "SDIO_D3CS" (at 215.9 92.71 0) (fields_autoplaced)
+    (effects (font (size 1.27 1.27)) (justify left bottom))
+  )
+  (label "SDIO_CMD" (at 215.9 82.55 0) (fields_autoplaced)
+    (effects (font (size 1.27 1.27)) (justify left bottom))
+  )
+  (label "DISPLAY_CS" (at 180.34 82.55 180) (fields_autoplaced)
+    (effects (font (size 1.27 1.27)) (justify right bottom))
+  )
   (label "I2C0_SDA" (at 25.4 43.18 180) (fields_autoplaced)
     (effects (font (size 1.27 1.27)) (justify right bottom))
   )
+  (label "TP_IRQ" (at 215.9 100.33 0) (fields_autoplaced)
+    (effects (font (size 1.27 1.27)) (justify left bottom))
+  )
+  (label "SPI1_SCK" (at 180.34 85.09 180) (fields_autoplaced)
+    (effects (font (size 1.27 1.27)) (justify right bottom))
+  )
+  (label "DISPLAY_BL" (at 180.34 87.63 180) (fields_autoplaced)
+    (effects (font (size 1.27 1.27)) (justify right bottom))
+  )
+  (label "SDIO_D0" (at 215.9 85.09 0) (fields_autoplaced)
+    (effects (font (size 1.27 1.27)) (justify left bottom))
+  )
   (label "I2C0_SCL" (at 35.56 40.64 180) (fields_autoplaced)
     (effects (font (size 1.27 1.27)) (justify right bottom))
   )
+  (label "DISPLAY_RST" (at 180.34 90.17 180) (fields_autoplaced)
+    (effects (font (size 1.27 1.27)) (justify right bottom))
+  )
+  (label "TP_CS" (at 215.9 97.79 0) (fields_autoplaced)
+    (effects (font (size 1.27 1.27)) (justify left bottom))
+  )
+  (label "DISPLAY_DC" (at 180.34 80.01 180) (fields_autoplaced)
+    (effects (font (size 1.27 1.27)) (justify right bottom))
+  )
   (symbol (lib_id "Device:R") (at 35.56 34.29 0) (unit 1)
     (in_bom yes) (on_board yes) (dnp no)
@@
       (effects (font (size 1.27 1.27)) (justify left))
     )
-    (property "Footprint" "Capacitor_SMD:C_0402_1005Metric" (at 33.782 34.29 90)
+    (property "Footprint" "Resistor_SMD:R_0402_1005Metric" (at 33.782 34.29 90)
       (effects (font (size 1.27 1.27)) hide)
     )
@@
     )
   )
+  (symbol (lib_id "Display_Graphic:Pico-ResTouch-LCD-2.8") (at 199.39 88.9 0) (unit 1)
+    (in_bom yes) (on_board yes) (dnp no) (fields_autoplaced)
+    (property "Reference" "U5" (at 199.39 104.14 0)
+      (effects (font (size 1.27 1.27)))
+    )
+    (property "Value" "~" (at 181.61 77.47 0)
+      (effects (font (size 1.27 1.27)))
+    )
+    (property "Footprint" "Display:Pico-ResTouch-LCD-2.8" (at 199.39 106.68 0)
+      (effects (font (size 1.27 1.27)) hide)
+    )
+    (property "Datasheet" "https://www.waveshare.com/wiki/Pico-ResTouch-LCD-2.8" (at 199.39 104.14 0)
+      (effects (font (size 1.27 1.27)) hide)
+    )
+    (pin "11")
+    (pin "21")
+    (pin "14")
+    (pin "24")
+    (pin "26")
+    (pin "27")
+    (pin "29")
+    (pin "3")
+    (pin "39")
+    (pin "7")
+    (pin "20")
+    (pin "15")
+    (pin "12")
+    (pin "22")
+    (pin "16")
+    (pin "25")
+    (pin "17")
+    (instances
+      (project "InternalPCBV2"
+        (path "/c0fadd27-a942-45e6-bb83-a446ca1e28e8/c45d2d52-0796-49f4-99c7-2a79c67462ab"
+          (reference "U5") (unit 1)
+        )
+      )
+    )
+  )
   (symbol (lib_id "power:+3.3V") (at 48.26 22.86 0) (unit 1)
     (in_bom yes) (on_board yes) (dnp no) (fields_autoplaced)
@@
       (effects (font (size 1.27 1.27)))
     )
-    (property "Footprint" "" (at 55.626 34.29 90)
+    (property "Footprint" "Battery:BatteryHolder_Keystone_103_1x20mm" (at 55.626 34.29 90)
       (effects (font (size 1.27 1.27)) hide)
     )
@@
     )
   )
+  (symbol (lib_id "power:GND") (at 198.12 76.2 0) (mirror x) (unit 1)
+    (in_bom yes) (on_board yes) (dnp no)
+    (property "Reference" "#PWR034" (at 198.12 69.85 0)
+      (effects (font (size 1.27 1.27)) hide)
+    )
+    (property "Value" "GND" (at 196.85 72.39 0)
+      (effects (font (size 1.27 1.27)))
+    )
+    (property "Footprint" "" (at 198.12 76.2 0)
+      (effects (font (size 1.27 1.27)) hide)
+    )
+    (property "Datasheet" "" (at 198.12 76.2 0)
+      (effects (font (size 1.27 1.27)) hide)
+    )
+    (pin "1")
+    (instances
+      (project "InternalPCBV2"
+        (path "/c0fadd27-a942-45e6-bb83-a446ca1e28e8/c45d2d52-0796-49f4-99c7-2a79c67462ab"
+          (reference "#PWR034") (unit 1)
+        )
+      )
+    )
+  )
+  (symbol (lib_id "power:+5V") (at 200.66 76.2 0) (unit 1)
+    (in_bom yes) (on_board yes) (dnp no)
+    (property "Reference" "#PWR035" (at 200.66 80.01 0)
+      (effects (font (size 1.27 1.27)) hide)
+    )
+    (property "Value" "+5V" (at 201.93 72.39 0)
+      (effects (font (size 1.27 1.27)))
+    )
+    (property "Footprint" "" (at 200.66 76.2 0)
+      (effects (font (size 1.27 1.27)) hide)
+    )
+    (property "Datasheet" "" (at 200.66 76.2 0)
+      (effects (font (size 1.27 1.27)) hide)
+    )
+    (pin "1")
+    (instances
+      (project "InternalPCBV2"
+        (path "/c0fadd27-a942-45e6-bb83-a446ca1e28e8/c45d2d52-0796-49f4-99c7-2a79c67462ab"
+          (reference "#PWR035") (unit 1)
+        )
+      )
+    )
+  )
   (symbol (lib_id "Device:R") (at 25.4 34.29 0) (unit 1)
     (in_bom yes) (on_board yes) (dnp no)
@@
       (effects (font (size 1.27 1.27)) (justify left))
     )
-    (property "Footprint" "Capacitor_SMD:C_0402_1005Metric" (at 23.622 34.29 90)
+    (property "Footprint" "Resistor_SMD:R_0402_1005Metric" (at 23.622 34.29 90)
       (effects (font (size 1.27 1.27)) hide)
     )
@@
       (effects (font (size 1.27 1.27)) (justify right))
     )
-    (property "Footprint" "Capacitor_SMD:C_0402_1005Metric" (at 67.818 54.61 90)
-      (effects (font (size 1.27 1.27)) hide)
-    )
+    (property "Footprint" "Resistor_SMD:R_0402_1005Metric" (at 67.818 54.61 90)
+      (effects (font (size 1.27 1.27)) hide)
+    )
